File: Hardware/Safe Cracker Shield.brd (EAGLE design)
At the start: 61 x 53.3 mm, 13 parts, among them J1 Zero Detect, J2 Power, J3 Current Sense, J4 Motor Control, J5 Motor Controller Output, J6 Motor Connect, J8 Handle Servo, U1 Arduino Uno

Commit message: Reorg file structure.
Parts:
- J1: value Zero Detect -> (none); device SparkFun-Connectors:JST-2-PTH -> SparkFun-Connectors:JST-3-PTH-VERT
- U$1: value SPARKX-LOGO4 -> SPARKX-LOGO5; device SparkX:SPARKX-MEDIUM -> SparkX:SPARKX-LARGE
- moved U$1 2.68 mm to (42.9, 20.4)
- moved J1 1.27 mm to (43.2, 12.7), turned to 0 degrees
Connections:
- removed net REED: J1.2, U1.D5
- new net PHOTO: J1.3, U1.D5
- net 5V: now also J1.1
- net GND: now also J1.2; no longer J1.1
- net PWM: now also U1.D6; no longer U1.D9
- net SERVO: now also U1.D9; no longer U1.D6
Routing:
- net PHOTO: track 0.00 -> 40.0 mm
- net REED: track 39.5 -> 0.00 mm
- net 5V: track 132.5 -> 147.7 mm
- net PWM: track 51.4 -> 63.6 mm
- net SERVO: track 78.7 -> 78.9 mm, vias 0 -> 1
Other:
- board text added: "N. Seidle"
- board text added: "Photo"
- board text removed: "Dial"
