File: Hardware/Safe Cracker Shield.brd (EAGLE design)
At the start: 61 x 53.3 mm, 15 parts, among them J2 Power, J3 Current Sense, J4 Motor Control, J5 Motor Controller Output, J6 Motor Connect, J8 Handle Servo, U1 Arduino Uno

Commit message: Fixed roll over indent count issue. Fixed net names on shield. Working version.
Connections:
- net CLOCK renamed DISPLAY_CLOCK
- net ENABLE renamed DISPLAY_LATCH
- net SER_OUT renamed DISPLAY_DATA
Changed lines of the file:
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@@
 <wire x1="25.4" y1="48.26" x2="24.13" y2="46.99" width="0.254" layer="16"/>
 </signal>
-<signal name="SER_OUT">
+<signal name="DISPLAY_DATA">
 <contactref element="J7" pad="4"/>
 <contactref element="U1" pad="A4"/>
 <wire x1="49.53" y1="5.08" x2="52.07" y2="2.54" width="0.254" layer="1"/>
 </signal>
-<signal name="ENABLE">
-<contactref element="J7" pad="3"/>
-<contactref element="U1" pad="A3"/>
-<wire x1="46.99" y1="5.08" x2="49.53" y2="2.54" width="0.254" layer="1"/>
-</signal>
-<signal name="CLOCK">
+<signal name="DISPLAY_CLOCK">
 <contactref element="J7" pad="2"/>
 <contactref element="U1" pad="A2"/>
@@
 <wire x1="36.83" y1="48.26" x2="34.29" y2="45.72" width="0.254" layer="1"/>
 </signal>
+<signal name="DISPLAY_LATCH">
+<contactref element="U1" pad="A3"/>
+<contactref element="J7" pad="3"/>
+<wire x1="46.99" y1="5.08" x2="49.53" y2="2.54" width="0.254" layer="1"/>
+</signal>
 </signals>

Commit message: Fixed net names on display. Clean up hardware directory.
Connections:
- net DISPLAY_CLOCK: now also J7.3, U1.A3; no longer J7.2, U1.A2
- net DISPLAY_LATCH: now also J7.2, U1.A2; no longer J7.3, U1.A3
Changed lines of the file:
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@@
 <wire x1="49.53" y1="5.08" x2="52.07" y2="2.54" width="0.254" layer="1"/>
-</signal>
-<signal name="DISPLAY_CLOCK">
-<contactref element="J7" pad="2"/>
-<contactref element="U1" pad="A2"/>
-<wire x1="44.45" y1="5.08" x2="46.99" y2="2.54" width="0.254" layer="1"/>
 </signal>
 <signal name="BUTTON">
@@
 </signal>
 <signal name="DISPLAY_LATCH">
+<contactref element="J7" pad="2"/>
+<contactref element="U1" pad="A2"/>
+<wire x1="44.45" y1="5.08" x2="46.99" y2="2.54" width="0.254" layer="1"/>
+</signal>
+<signal name="DISPLAY_CLOCK">
+<contactref element="J7" pad="3"/>
 <contactref element="U1" pad="A3"/>
-<contactref element="J7" pad="3"/>
 <wire x1="46.99" y1="5.08" x2="49.53" y2="2.54" width="0.254" layer="1"/>
 </signal>
