File: Hardware/Safe Cracker Shield.sch (EAGLE design)
At the start: 13 parts, among them J1 Zero Detect, J2 Power, J3 Current Sense, J4 Motor Control, J5 Motor Controller Output, J6 Motor Connect, J8 Handle Servo, U1 Arduino Uno

Commit message: Reorg file structure.
Parts:
- J1: value Zero Detect -> (none); device SparkFun-Connectors:CONN_02JST-PTH-2 -> SparkFun-Connectors:CONN_03JST-PTH-VERT
- U$1: value SPARKX-LOGO4 -> SPARKX-LOGO5; device SparkX:SPARKX-LOGO4 -> SparkX:SPARKX-LOGO5
Connections:
- removed net REED: J1.2, U1.*D5
- new net PHOTO: J1.3, U1.*D5
- net 5V: now also J1.1
- net GND: now also J1.2; no longer J1.1
- net PWM: now also U1.*D6; no longer U1.*D9
- net SERVO: now also U1.*D9; no longer U1.*D6
