File: Hardware/Safe Cracker Shield.sch (EAGLE design)
At the start: 15 parts, among them J2 Power, J3 Current Sense, J4 Motor Control, J5 Motor Controller Output, J6 Motor Connect, J8 Handle Servo, U1 Arduino Uno

Commit message: Fixed roll over indent count issue. Fixed net names on shield. Working version.
Connections:
- net CLOCK renamed DISPLAY_CLOCK
- net ENABLE renamed DISPLAY_LATCH
- net SER_OUT renamed DISPLAY_DATA
Changed lines of the file:
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@@
 </segment>
 </net>
-<net name="SER_OUT" class="0">
+<net name="DISPLAY_DATA" class="0">
 <segment>
 <pinref part="J7" gate="G$1" pin="4"/>
@@
 </segment>
 </net>
-<net name="ENABLE" class="0">
-<segment>
-<pinref part="J7" gate="G$1" pin="3"/>
-<wire x1="210.82" y1="109.22" x2="213.36" y2="109.22" width="0.1524" layer="91"/>
-<label x="213.36" y="109.22" size="1.27" layer="95" xref="yes"/>
-</segment>
-<segment>
-<pinref part="U1" gate="G$1" pin="A3"/>
-<wire x1="43.18" y1="160.02" x2="40.64" y2="160.02" width="0.1524" layer="91"/>
-<label x="40.64" y="160.02" size="1.27" layer="95" rot="R180" xref="yes"/>
-</segment>
-</net>
-<net name="CLOCK" class="0">
+<net name="DISPLAY_CLOCK" class="0">
 <segment>
 <pinref part="J7" gate="G$1" pin="2"/>
@@
 </segment>
 </net>
+<net name="DISPLAY_LATCH" class="0">
+<segment>
+<pinref part="U1" gate="G$1" pin="A3"/>
+<wire x1="43.18" y1="160.02" x2="40.64" y2="160.02" width="0.1524" layer="91"/>
+<label x="40.64" y="160.02" size="1.27" layer="95" rot="R180" xref="yes"/>
+</segment>
+<segment>
+<pinref part="J7" gate="G$1" pin="3"/>
+<wire x1="210.82" y1="109.22" x2="213.36" y2="109.22" width="0.1524" layer="91"/>
+<label x="213.36" y="109.22" size="1.27" layer="95" xref="yes"/>
+</segment>
+</net>

Commit message: Fixed net names on display. Clean up hardware directory.
Connections:
- net DISPLAY_CLOCK: now also J7.3, U1.A3; no longer J7.2, U1.A2
- net DISPLAY_LATCH: now also J7.2, U1.A2; no longer J7.3, U1.A3
Changed lines of the file:
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@@
-</segment>
-</net>
-<net name="DISPLAY_CLOCK" class="0">
-<segment>
-<pinref part="J7" gate="G$1" pin="2"/>
-<wire x1="210.82" y1="106.68" x2="213.36" y2="106.68" width="0.1524" layer="91"/>
-<label x="213.36" y="106.68" size="1.27" layer="95" xref="yes"/>
-</segment>
-<segment>
-<pinref part="U1" gate="G$1" pin="A2"/>
-<wire x1="43.18" y1="162.56" x2="40.64" y2="162.56" width="0.1524" layer="91"/>
-<label x="40.64" y="162.56" size="1.27" layer="95" rot="R180" xref="yes"/>
 </segment>
 </net>
@@
 <net name="DISPLAY_LATCH" class="0">
 <segment>
-<pinref part="U1" gate="G$1" pin="A3"/>
-<wire x1="43.18" y1="160.02" x2="40.64" y2="160.02" width="0.1524" layer="91"/>
-<label x="40.64" y="160.02" size="1.27" layer="95" rot="R180" xref="yes"/>
+<pinref part="J7" gate="G$1" pin="2"/>
+<wire x1="210.82" y1="106.68" x2="213.36" y2="106.68" width="0.1524" layer="91"/>
+<label x="213.36" y="106.68" size="1.27" layer="95" xref="yes"/>
 </segment>
+<segment>
+<pinref part="U1" gate="G$1" pin="A2"/>
+<wire x1="43.18" y1="162.56" x2="40.64" y2="162.56" width="0.1524" layer="91"/>
+<label x="40.64" y="162.56" size="1.27" layer="95" rot="R180" xref="yes"/>
+</segment>
+</net>
+<net name="DISPLAY_CLOCK" class="0">
 <segment>
 <pinref part="J7" gate="G$1" pin="3"/>
@@
 <label x="213.36" y="109.22" size="1.27" layer="95" xref="yes"/>
 </segment>
+<segment>
+<pinref part="U1" gate="G$1" pin="A3"/>
+<wire x1="43.18" y1="160.02" x2="40.64" y2="160.02" width="0.1524" layer="91"/>
+<label x="40.64" y="160.02" size="1.27" layer="95" rot="R180" xref="yes"/>
+</segment>
 </net>
